Commit message: Update path to correct package name

File: webots_rosconfr/resource/TT02_jaune.urdf (robot description, URDF)
Before this commit: robot yellow_car, 8 links, 7 joints
Links:
- link base_link: geometry visual mesh filename=package://webots_rosconfr/protos/ChevroletCamaroLight.stl

File: webots_rosconfr/resource/TT02_jaune_cam.urdf (robot description, URDF)
Before this commit: robot yellow_car, 9 links, 8 joints
Links:
- link base_link: geometry visual mesh filename=package://webots_rosconfr/protos/ChevroletCamaroLight.stl
